File: zyypadmarco.kicad_sch (KiCad schematic)
At the start: 0 parts

Commit message: schematic
Parts:
- added C1, C2: 30pf, symbol Device:C_Small
- added C10, C17, C3, C4, C5: 1u, Capacitor_SMD:C_0402_1005Metric, symbol Device:C_Small
- added C11, C12, C13, C14, C15, C16, C6, C7, C8, C9: 100n, Capacitor_SMD:C_0402_1005Metric, symbol Device:C_Small
- added F1: 700mA, Fuse:Fuse_0402_1005Metric, symbol Device:Polyfuse_Small
- added FB1: 100 Ohm @ 100 MHz, Inductor_SMD:L_0402_1005Metric, symbol Device:FerriteBead_Small
- added J1: USB_C_Receptacle_USB2.0_16P, symbol Connector:USB_C_Receptacle_USB2.0_16P
- added J2: JST - 1.00mm 4 Pin, Connector_JST:JST_SH_SM04B-SRSS-TB_1x04-1MP_P1.00mm_Horizontal, symbol Connector_Generic_MountingPin:Conn_01x04_MountingPin
- added R1: 1k, symbol Device:R_Small
- added R2, R3: 5.1k, symbol Device:R_Small
- added R4, R5: 22, symbol Device:R_Small
- added SW22, SW23: button, symbol Switch:SW_Push
- added U1: RP2040, Package_DFN_QFN:QFN-56-1EP_7x7mm_P0.4mm_EP3.2x3.2mm, symbol MCU_RaspberryPi:RP2040
- added U3: USBLC6-2SC6, Package_TO_SOT_SMD:SOT-23-6, symbol Power_Protection:USBLC6-2SC6
- added U4: 3.3V Fixed Regulator, Package_TO_SOT_SMD:TSOT-23, symbol Regulator_Linear:AP2127N3-1.2
- added U5: ZD25D40CNJGR, USON8:USON-8_1.5x1.5mm_P0.45mm, symbol Flash_NOR_SPI:ZD25D40CNJGR
- added Y1: 12Mhz 3225, symbol Device:Crystal_GND24_Small
Connections:
- new net: C3.1, U4.2 (VO)
- new net: F1.1, FB1.1
- new net: R5.2, U1.47 (USB_DP)
- new net: R1.1, U1.21 (XOUT)
- new net: C4.2, U4.3 (VI)
- new net: J1.A5 (CC1), R3.2
- new net: R4.1, U1.46 (USB_DM)
- new net: J1.B5 (CC2), R2.2
- new net +1V1: C16.1, C5.2, C6.1, U1.23 (DVDD), U1.45 (VREG_VOUT), U1.50 (DVDD)
- new net +3.3V: C1.2, C10.1, C10.2, C11.1, C11.2, C12.1, C12.2, C13.1, C13.2, C14.1, C14.2, C15.1, C15.2, C16.2, C17.1, C17.2, C2.2, C3.2, C4.1, C5.1, C6.2, C7.1, C7.2, C8.1, C8.2, C9.1, C9.2, FB1.2, J1.A1 (GND), J1.A12 (GND), J1.B1 (GND), J1.B12 (GND), J2.1 (Pin_1), J2.4 (Pin_4), J2.MP (MountPin), R2.1, R3.1, SW22.1, SW23.1, U1.1 (IOVDD), U1.10 (IOVDD), U1.19 (TESTEN), U1.22 (IOVDD), U1.33 (IOVDD), U1.42 (IOVDD), U1.43 (ADC_AVDD), U1.44 (VREG_IN), U1.48 (USB_VDD), U1.49 (IOVDD), U1.57 (GND), U3.2 (GND), U4.1 (GND), U5.4 (V_{SS}), U5.8 (V_{CC}), U5.9 (PAD/V_{SS}), Y1.2, Y1.4
- new net CS: SW22.2, U1.56 (QSPI_SS), U5.1 (~{CS})
- new net D1+: J1.A6 (D+), J1.B6 (D+), U3.4 (I/O2)
- new net D1-: J1.A7 (D-), J1.B7 (D-), U3.6 (I/O1)
- new net DN: J2.2 (Pin_2), R4.2, U3.1 (I/O1)
- new net DP: J2.3 (Pin_3), R5.1, U3.3 (I/O2)
- new net RUN: SW23.2, U1.26 (RUN)
- new net SCLK: U1.52 (QSPI_SCLK), U5.6 (SCLK)
- new net SD0: U1.53 (QSPI_SD0), U5.5 (MOSI/D0)
- new net SD1: U1.55 (QSPI_SD1), U5.2 (MISO/D1)
- new net SD2: U1.54 (QSPI_SD2), U5.3 (~{WP})
- new net VBUS: F1.2, J1.A4 (VBUS), J1.A9 (VBUS), J1.B4 (VBUS), J1.B9 (VBUS), U3.5 (VBUS)
- new net Xin: C2.1, U1.20 (XIN), Y1.3
- new net Xout: C1.1, R1.2, Y1.1
- no-connect marks 0 -> 3
Other:
- added sheet matrix (untitled.kicad_sch)
- note added: "Crystal"
- note added: "Marvel Cinematic Universe"
- note added: "Memory"
- note added: "USB-C + JST"
- note added: "power manager"

Commit message: pcb
Parts:
- C16: renamed from C2; footprint (none) -> Capacitor_SMD:C_0402_1005Metric
- C17: renamed from C1; footprint (none) -> Capacitor_SMD:C_0402_1005Metric
- J1: footprint (none) -> Connector_USB:USB_C_Receptacle_GCT_USB4110
- PS1: renamed from SW23; footprint (none) -> Button_Switch_SMD:SW_Push_1P1T_NO_E-Switch_TL3301NxxxxxG
- PS2: renamed from SW22; footprint (none) -> Button_Switch_SMD:SW_Push_1P1T_NO_E-Switch_TL3301NxxxxxG
- R1: renamed from R5; footprint (none) -> Resistor_SMD:R_0805_2012Metric
- R2: renamed from R4; footprint (none) -> Resistor_SMD:R_0805_2012Metric
- R3: renamed from R1; footprint (none) -> Resistor_SMD:R_0805_2012Metric
- R4: renamed from R2; footprint (none) -> Resistor_SMD:R_0805_2012Metric
- R5: renamed from R3; footprint (none) -> Resistor_SMD:R_0805_2012Metric
- Y1: footprint (none) -> Crystal:Crystal_SMD_3225-4Pin_3.2x2.5mm_HandSoldering
- renumbered C17 to C1, C12 to C10, C3 to C11, C6 to C12, C7 to C2, C8 to C3, C9 to C4, C10 to C5, C11 to C6, C4 to C7, C5 to C8, C16 to C9, U3 to U2, U5 to U3
